File: Kicad_JE_SteinerVCF/_saved_JE-SMD-SteinerVCF.sch (KiCad schematic (older format))
At the start: 49 parts, among them J201 HP, J202 BP, J203 LP, J204 Out, J205 CV, P201 Doepfer_Power_10pin, Q201 MMBT2907A, Q202 MMBT2222A, Q203 MMBT2222A, Q204 MMBT2222A

Commit message: Place SMD init
Parts:
- C201: value C -> 100n; footprint Capacitor_SMD:C_0603_1608Metric_Pad1.05x0.95mm_HandSolder -> Capacitor_SMD:C_0805_2012Metric_Pad1.15x1.40mm_HandSolder
- C202, C205: value CP -> 100uF; footprint Capacitor_THT:CP_Radial_D10.0mm_P5.00mm -> Capacitor_Tantalum_SMD:CP_EIA-7343-15_Kemet-W_Pad2.25x2.55mm_HandSolder
- C204, C206, C207, C208, C209, C210: footprint Capacitor_SMD:C_0603_1608Metric_Pad1.05x0.95mm_HandSolder -> Capacitor_SMD:C_0805_2012Metric_Pad1.15x1.40mm_HandSolder
- RV202, RV203: footprint Potentiometer_THT:Potentiometer_Alps_RK09K_Single_Vertical -> Potentiometer_THT:Potentiometer_Piher_PT-6-V_Vertical
Changed lines of the file:
@@
 AR Path="/5C4E0953/5C4E61A4" Ref="C201"  Part="1"
 F 0 "C201" H 2665 1096 50  0000 L CNN
-F 1 "C" H 2665 1005 50  0000 L CNN
-F 2 "Capacitor_SMD:C_0603_1608Metric_Pad1.05x0.95mm_HandSolder" H 2588 900 50  0001 C CNN
+F 1 "100n" H 2665 1005 50  0000 L CNN
+F 2 "Capacitor_SMD:C_0805_2012Metric_Pad1.15x1.40mm_HandSolder" H 2588 900 50  0001 C CNN
 F 3 "~" H 2550 1050 50  0001 C CNN
 	1    2550 1050
@@
 F 0 "C204" H 4015 1096 50  0000 L CNN
 F 1 "100nF" H 4015 1005 50  0000 L CNN
-F 2 "Capacitor_SMD:C_0603_1608Metric_Pad1.05x0.95mm_HandSolder" H 3938 900 50  0001 C CNN
+F 2 "Capacitor_SMD:C_0805_2012Metric_Pad1.15x1.40mm_HandSolder" H 3938 900 50  0001 C CNN
 F 3 "~" H 3900 1050 50  0001 C CNN
 	1    3900 1050
@@
 AR Path="/5C4E0953/5C4E61B2" Ref="C202"  Part="1"
 F 0 "C202" H 3118 1096 50  0000 L CNN
-F 1 "CP" H 3118 1005 50  0000 L CNN
-F 2 "Capacitor_THT:CP_Radial_D10.0mm_P5.00mm" H 3038 900 50  0001 C CNN
+F 1 "100uF" H 3118 1005 50  0000 L CNN
+F 2 "Capacitor_Tantalum_SMD:CP_EIA-7343-15_Kemet-W_Pad2.25x2.55mm_HandSolder" H 3038 900 50  0001 C CNN
 F 3 "~" H 3000 1050 50  0001 C CNN
 	1    3000 1050
@@
 F 0 "C209" H 3665 5996 50  0000 L CNN
 F 1 "4n7" H 3665 5905 50  0000 L CNN
-F 2 "Capacitor_SMD:C_0603_1608Metric_Pad1.05x0.95mm_HandSolder" H 3588 5800 50  0001 C CNN
+F 2 "Capacitor_SMD:C_0805_2012Metric_Pad1.15x1.40mm_HandSolder" H 3588 5800 50  0001 C CNN
 F 3 "~" H 3550 5950 50  0001 C CNN
 	1    3550 5950
@@
 F 0 "C208" H 2965 5996 50  0000 L CNN
 F 1 "4n7" H 2965 5905 50  0000 L CNN
-F 2 "Capacitor_SMD:C_0603_1608Metric_Pad1.05x0.95mm_HandSolder" H 2888 5800 50  0001 C CNN
+F 2 "Capacitor_SMD:C_0805_2012Metric_Pad1.15x1.40mm_HandSolder" H 2888 5800 50  0001 C CNN
 F 3 "~" H 2850 5950 50  0001 C CNN
 	1    2850 5950
@@
 F 0 "C210" H 4315 5996 50  0000 L CNN
 F 1 "4n7" H 4315 5905 50  0000 L CNN
-F 2 "Capacitor_SMD:C_0603_1608Metric_Pad1.05x0.95mm_HandSolder" H 4238 5800 50  0001 C CNN
+F 2 "Capacitor_SMD:C_0805_2012Metric_Pad1.15x1.40mm_HandSolder" H 4238 5800 50  0001 C CNN
 F 3 "~" H 4200 5950 50  0001 C CNN
 	1    4200 5950
@@
 F 0 "RV202" V 1393 5750 50  0000 C CNN
 F 1 "500k" V 1484 5750 50  0000 C CNN
-F 2 "Potentiometer_THT:Potentiometer_Alps_RK09K_Single_Vertical" H 1600 5750 50  0001 C CNN
+F 2 "Potentiometer_THT:Potentiometer_Piher_PT-6-V_Vertical" H 1600 5750 50  0001 C CNN
 F 3 "~" H 1600 5750 50  0001 C CNN
 	1    1600 5750
@@
 F 0 "RV203" H 1130 6796 50  0000 R CNN
 F 1 "25k" H 1130 6705 50  0000 R CNN
-F 2 "Potentiometer_THT:Potentiometer_Alps_RK09K_Single_Vertical" H 1200 6750 50  0001 C CNN
+F 2 "Potentiometer_THT:Potentiometer_Piher_PT-6-V_Vertical" H 1200 6750 50  0001 C CNN
 F 3 "~" H 1200 6750 50  0001 C CNN
 	1    1200 6750
@@
 F 0 "C206" V 2448 2500 50  0000 C CNN
 F 1 "1u" V 2539 2500 50  0000 C CNN
-F 2 "Capacitor_SMD:C_0603_1608Metric_Pad1.05x0.95mm_HandSolder" H 2738 2350 50  0001 C CNN
+F 2 "Capacitor_SMD:C_0805_2012Metric_Pad1.15x1.40mm_HandSolder" H 2738 2350 50  0001 C CNN
 F 3 "~" H 2700 2500 50  0001 C CNN
 	1    2700 2500
@@
 F 0 "C207" V 4905 2600 50  0000 C CNN
 F 1 "10u" V 4814 2600 50  0000 C CNN
-F 2 "Capacitor_SMD:C_0603_1608Metric_Pad1.05x0.95mm_HandSolder" H 4688 2450 50  0001 C CNN
+F 2 "Capacitor_SMD:C_0805_2012Metric_Pad1.15x1.40mm_HandSolder" H 4688 2450 50  0001 C CNN
 F 3 "~" H 4650 2600 50  0001 C CNN
 	1    4650 2600
@@
 AR Path="/5C4E0953/5C59B140" Ref="C205"  Part="1"
 F 0 "C205" V 1355 1400 50  0000 C CNN
-F 1 "CP" V 1264 1400 50  0000 C CNN
-F 2 "Capacitor_THT:CP_Radial_D10.0mm_P5.00mm" H 1138 1250 50  0001 C CNN
+F 1 "100uF" V 1264 1400 50  0000 C CNN
+F 2 "Capacitor_Tantalum_SMD:CP_EIA-7343-15_Kemet-W_Pad2.25x2.55mm_HandSolder" H 1138 1250 50  0001 C CNN
 F 3 "~" H 1100 1400 50  0001 C CNN
 	1    1100 1400
