File: Kicad_JE_SteinerVCF/_saved_Kicad_JE_SteinerVCF.sch (KiCad schematic (older format))
At the start: 49 parts, among them J101 AudioJack2_SwitchT, J102 AudioJack2_SwitchT, J103 AudioJack2_SwitchT, J104 AudioJack2_SwitchT, J105 AudioJack2_SwitchT, P101 Doepfer_Power_10pin, Q101 BC559, Q102 BC549, Q103 BC549, Q104 BC549

Commit message: THT update - minor
Parts:
- J101: value AudioJack2_SwitchT -> HP
- J102: value AudioJack2_SwitchT -> BP
- J103: value AudioJack2_SwitchT -> LP
- J104: value AudioJack2_SwitchT -> Out
- J105: value AudioJack2_SwitchT -> CV
Changed lines of the file:
@@
 P 950 1900
 F 0 "J101" H 980 2225 50  0000 C CNN
-F 1 "AudioJack2_SwitchT" H 980 2134 50  0000 C CNN
+F 1 "HP" H 980 2134 50  0000 C CNN
 F 2 "AJ-Dropbox-Kicad:PJ301SM" H 950 1900 50  0001 C CNN
 F 3 "~" H 950 1900 50  0001 C CNN
@@
 P 950 2300
 F 0 "J102" H 980 2625 50  0000 C CNN
-F 1 "AudioJack2_SwitchT" H 980 2534 50  0000 C CNN
+F 1 "BP" H 980 2534 50  0000 C CNN
 F 2 "AJ-Dropbox-Kicad:PJ301SM" H 950 2300 50  0001 C CNN
 F 3 "~" H 950 2300 50  0001 C CNN
@@
 P 950 2750
 F 0 "J103" H 980 3075 50  0000 C CNN
-F 1 "AudioJack2_SwitchT" H 980 2984 50  0000 C CNN
+F 1 "LP" H 980 2984 50  0000 C CNN
 F 2 "AJ-Dropbox-Kicad:PJ301SM" H 950 2750 50  0001 C CNN
 F 3 "~" H 950 2750 50  0001 C CNN
@@
 P 950 3200
 F 0 "J104" H 980 3525 50  0000 C CNN
-F 1 "AudioJack2_SwitchT" H 980 3434 50  0000 C CNN
+F 1 "Out" H 980 3434 50  0000 C CNN
 F 2 "AJ-Dropbox-Kicad:PJ301SM" H 950 3200 50  0001 C CNN
 F 3 "~" H 950 3200 50  0001 C CNN
@@
 P 950 3600
 F 0 "J105" H 980 3925 50  0000 C CNN
-F 1 "AudioJack2_SwitchT" H 980 3834 50  0000 C CNN
+F 1 "CV" H 980 3834 50  0000 C CNN
 F 2 "AJ-Dropbox-Kicad:PJ301SM" H 950 3600 50  0001 C CNN
 F 3 "~" H 950 3600 50  0001 C CNN
