File: Kicad_JE_SteinerVCF/JE-SMD-SteinerVCF.sch (KiCad schematic (older format))
At the start: 49 parts

Commit message: ERC, Footprints and Annotation in SCH
Parts:
- C201, C204, C206, C207, C208, C209, C210: renamed from C?; footprint (none) -> Capacitor_SMD:C_0603_1608Metric_Pad1.05x0.95mm_HandSolder
- C202, C203, C205, C211: renamed from C?; footprint (none) -> Capacitor_THT:CP_Radial_D10.0mm_P5.00mm
- J201, J202, J203, J204, J205: renamed from J?; footprint (none) -> AJ-Dropbox-Kicad:PJ301SM
- Q201: renamed from Q?; footprint (none) -> Active:SOT-23-3
- Q202, Q203, Q204: renamed from Q?; footprint SOT23 -> Active:SOT-23-3
- R201, R202, R203, R204, R205, R206, R207, R208, R209, R210, R211, R212, R213, R214, R215, R216, R217: renamed from R?; footprint (none) -> Resistor_SMD:R_0805_2012Metric_Pad1.15x1.40mm_HandSolder
- RV201, RV202, RV203: renamed from RV?; footprint (none) -> Potentiometer_THT:Potentiometer_Alps_RK09K_Single_Vertical
- gave numbers to parts that had none: 9
Connections:
- wire segments 162 -> 158

Commit message: Net - names conn
Parts:
- J201: value AudioJack2_SwitchT -> HP
- J202: value AudioJack2_SwitchT -> BP
- J203: value AudioJack2_SwitchT -> LP
- J204: value AudioJack2_SwitchT -> Out
- J205: value AudioJack2_SwitchT -> CV
- Q201: symbol MMBT2907A:MMBT2907A -> MMBT2907_:MMBT2907*
Changed lines of the file:
@@
 AR Path="/5C4E0953/5C4E632A" Ref="J201"  Part="1"
 F 0 "J201" H 1130 2275 50  0000 C CNN
-F 1 "AudioJack2_SwitchT" H 1130 2184 50  0000 C CNN
+F 1 "HP" H 1130 2184 50  0000 C CNN
 F 2 "AJ-Dropbox-Kicad:PJ301SM" H 1100 1950 50  0001 C CNN
 F 3 "~" H 1100 1950 50  0001 C CNN
@@
 AR Path="/5C4E0953/5C4E6331" Ref="J202"  Part="1"
 F 0 "J202" H 1130 2675 50  0000 C CNN
-F 1 "AudioJack2_SwitchT" H 1130 2584 50  0000 C CNN
+F 1 "BP" H 1130 2584 50  0000 C CNN
 F 2 "AJ-Dropbox-Kicad:PJ301SM" H 1100 2350 50  0001 C CNN
 F 3 "~" H 1100 2350 50  0001 C CNN
@@
 AR Path="/5C4E0953/5C4E6338" Ref="J203"  Part="1"
 F 0 "J203" H 1130 3125 50  0000 C CNN
-F 1 "AudioJack2_SwitchT" H 1130 3034 50  0000 C CNN
+F 1 "LP" H 1130 3034 50  0000 C CNN
 F 2 "AJ-Dropbox-Kicad:PJ301SM" H 1100 2800 50  0001 C CNN
 F 3 "~" H 1100 2800 50  0001 C CNN
@@
 AR Path="/5C4E0953/5C4E635B" Ref="J204"  Part="1"
 F 0 "J204" H 1130 3575 50  0000 C CNN
-F 1 "AudioJack2_SwitchT" H 1130 3484 50  0000 C CNN
+F 1 "Out" H 1130 3484 50  0000 C CNN
 F 2 "AJ-Dropbox-Kicad:PJ301SM" H 1100 3250 50  0001 C CNN
 F 3 "~" H 1100 3250 50  0001 C CNN
@@
 AR Path="/5C4E0953/5C4E6362" Ref="J205"  Part="1"
 F 0 "J205" H 1130 3975 50  0000 C CNN
-F 1 "AudioJack2_SwitchT" H 1130 3884 50  0000 C CNN
+F 1 "CV" H 1130 3884 50  0000 C CNN
 F 2 "AJ-Dropbox-Kicad:PJ301SM" H 1100 3650 50  0001 C CNN
 F 3 "~" H 1100 3650 50  0001 C CNN
@@
 	1800 6150 1950 6150
 $Comp
-L MMBT2907A:MMBT2907A Q201
+L MMBT2907_:MMBT2907* Q201
 U 1 1 5C5E7BD8
 P 4300 2200

Commit message: Place SMD init
Parts:
- C201, C204, C206, C207, C208, C209, C210: footprint Capacitor_SMD:C_0603_1608Metric_Pad1.05x0.95mm_HandSolder -> Capacitor_SMD:C_0805_2012Metric_Pad1.15x1.40mm_HandSolder
- C202, C205: footprint Capacitor_THT:CP_Radial_D10.0mm_P5.00mm -> Capacitor_Tantalum_SMD:CP_EIA-7343-15_Kemet-W_Pad2.25x2.55mm_HandSolder
- RV202, RV203: footprint Potentiometer_THT:Potentiometer_Alps_RK09K_Single_Vertical -> Potentiometer_THT:Potentiometer_Piher_PT-6-V_Vertical
Changed lines of the file:
@@
 F 0 "C201" H 2665 1096 50  0000 L CNN
 F 1 "C" H 2665 1005 50  0000 L CNN
-F 2 "Capacitor_SMD:C_0603_1608Metric_Pad1.05x0.95mm_HandSolder" H 2588 900 50  0001 C CNN
+F 2 "Capacitor_SMD:C_0805_2012Metric_Pad1.15x1.40mm_HandSolder" H 2588 900 50  0001 C CNN
 F 3 "~" H 2550 1050 50  0001 C CNN
 	1    2550 1050
@@
 F 0 "C204" H 4015 1096 50  0000 L CNN
 F 1 "100nF" H 4015 1005 50  0000 L CNN
-F 2 "Capacitor_SMD:C_0603_1608Metric_Pad1.05x0.95mm_HandSolder" H 3938 900 50  0001 C CNN
+F 2 "Capacitor_SMD:C_0805_2012Metric_Pad1.15x1.40mm_HandSolder" H 3938 900 50  0001 C CNN
 F 3 "~" H 3900 1050 50  0001 C CNN
 	1    3900 1050
@@
 F 0 "C202" H 3118 1096 50  0000 L CNN
 F 1 "CP" H 3118 1005 50  0000 L CNN
-F 2 "Capacitor_THT:CP_Radial_D10.0mm_P5.00mm" H 3038 900 50  0001 C CNN
+F 2 "Capacitor_Tantalum_SMD:CP_EIA-7343-15_Kemet-W_Pad2.25x2.55mm_HandSolder" H 3038 900 50  0001 C CNN
 F 3 "~" H 3000 1050 50  0001 C CNN
 	1    3000 1050
@@
 F 0 "C209" H 3665 5996 50  0000 L CNN
 F 1 "4n7" H 3665 5905 50  0000 L CNN
-F 2 "Capacitor_SMD:C_0603_1608Metric_Pad1.05x0.95mm_HandSolder" H 3588 5800 50  0001 C CNN
+F 2 "Capacitor_SMD:C_0805_2012Metric_Pad1.15x1.40mm_HandSolder" H 3588 5800 50  0001 C CNN
 F 3 "~" H 3550 5950 50  0001 C CNN
 	1    3550 5950
@@
 F 0 "C208" H 2965 5996 50  0000 L CNN
 F 1 "4n7" H 2965 5905 50  0000 L CNN
-F 2 "Capacitor_SMD:C_0603_1608Metric_Pad1.05x0.95mm_HandSolder" H 2888 5800 50  0001 C CNN
+F 2 "Capacitor_SMD:C_0805_2012Metric_Pad1.15x1.40mm_HandSolder" H 2888 5800 50  0001 C CNN
 F 3 "~" H 2850 5950 50  0001 C CNN
 	1    2850 5950
@@
 F 0 "C210" H 4315 5996 50  0000 L CNN
 F 1 "4n7" H 4315 5905 50  0000 L CNN
-F 2 "Capacitor_SMD:C_0603_1608Metric_Pad1.05x0.95mm_HandSolder" H 4238 5800 50  0001 C CNN
+F 2 "Capacitor_SMD:C_0805_2012Metric_Pad1.15x1.40mm_HandSolder" H 4238 5800 50  0001 C CNN
 F 3 "~" H 4200 5950 50  0001 C CNN
 	1    4200 5950
@@
 F 0 "RV202" V 1393 5750 50  0000 C CNN
 F 1 "500k" V 1484 5750 50  0000 C CNN
-F 2 "Potentiometer_THT:Potentiometer_Alps_RK09K_Single_Vertical" H 1600 5750 50  0001 C CNN
+F 2 "Potentiometer_THT:Potentiometer_Piher_PT-6-V_Vertical" H 1600 5750 50  0001 C CNN
 F 3 "~" H 1600 5750 50  0001 C CNN
 	1    1600 5750
@@
 F 0 "RV203" H 1130 6796 50  0000 R CNN
 F 1 "25k" H 1130 6705 50  0000 R CNN
-F 2 "Potentiometer_THT:Potentiometer_Alps_RK09K_Single_Vertical" H 1200 6750 50  0001 C CNN
+F 2 "Potentiometer_THT:Potentiometer_Piher_PT-6-V_Vertical" H 1200 6750 50  0001 C CNN
 F 3 "~" H 1200 6750 50  0001 C CNN
 	1    1200 6750
@@
 F 0 "C206" V 2448 2500 50  0000 C CNN
 F 1 "1u" V 2539 2500 50  0000 C CNN
-F 2 "Capacitor_SMD:C_0603_1608Metric_Pad1.05x0.95mm_HandSolder" H 2738 2350 50  0001 C CNN
+F 2 "Capacitor_SMD:C_0805_2012Metric_Pad1.15x1.40mm_HandSolder" H 2738 2350 50  0001 C CNN
 F 3 "~" H 2700 2500 50  0001 C CNN
 	1    2700 2500
@@
 F 0 "C207" V 4905 2600 50  0000 C CNN
 F 1 "10u" V 4814 2600 50  0000 C CNN
-F 2 "Capacitor_SMD:C_0603_1608Metric_Pad1.05x0.95mm_HandSolder" H 4688 2450 50  0001 C CNN
+F 2 "Capacitor_SMD:C_0805_2012Metric_Pad1.15x1.40mm_HandSolder" H 4688 2450 50  0001 C CNN
 F 3 "~" H 4650 2600 50  0001 C CNN
 	1    4650 2600
@@
 F 0 "C205" V 1355 1400 50  0000 C CNN
 F 1 "CP" V 1264 1400 50  0000 C CNN
-F 2 "Capacitor_THT:CP_Radial_D10.0mm_P5.00mm" H 1138 1250 50  0001 C CNN
+F 2 "Capacitor_Tantalum_SMD:CP_EIA-7343-15_Kemet-W_Pad2.25x2.55mm_HandSolder" H 1138 1250 50  0001 C CNN
 F 3 "~" H 1100 1400 50  0001 C CNN
 	1    1100 1400

Commit message: SMD section routed RevA
Parts:
- C201: value C -> 100n
- C202, C205: value CP -> 100uF
Connections:
- net labels added: BP2, CV2, FilterOut2, HP2, LP2, Out2
- net labels removed: BP, CV, FilterOut, HP, LP, Out
- wire segments 158 -> 160
Changed lines of the file:
@@
 AR Path="/5C4E0953/5C4E61A4" Ref="C201"  Part="1"
 F 0 "C201" H 2665 1096 50  0000 L CNN
-F 1 "C" H 2665 1005 50  0000 L CNN
+F 1 "100n" H 2665 1005 50  0000 L CNN
 F 2 "Capacitor_SMD:C_0805_2012Metric_Pad1.15x1.40mm_HandSolder" H 2588 900 50  0001 C CNN
 F 3 "~" H 2550 1050 50  0001 C CNN
@@
 AR Path="/5C4E0953/5C4E61B2" Ref="C202"  Part="1"
 F 0 "C202" H 3118 1096 50  0000 L CNN
-F 1 "CP" H 3118 1005 50  0000 L CNN
+F 1 "100uF" H 3118 1005 50  0000 L CNN
 F 2 "Capacitor_Tantalum_SMD:CP_EIA-7343-15_Kemet-W_Pad2.25x2.55mm_HandSolder" H 3038 900 50  0001 C CNN
 F 3 "~" H 3000 1050 50  0001 C CNN
@@
 	2850 6350 2850 6100
 Text GLabel 3500 6200 0    59   Input ~ 12
-HP
+HP2
 Text GLabel 2700 6350 0    59   Input ~ 12
-BP
+BP2
 Wire Wire Line
 	3500 6200 3550 6200
@@
 	2150 4900 2150 5050
 Text GLabel 2050 4900 0    59   Input ~ 12
-LP
+LP2
 Wire Wire Line
 	2050 4900 2150 4900
@@
 	1750 6150 1800 6150
 Text GLabel 1300 6150 0    59   Input ~ 12
-CV
+CV2
 Wire Wire Line
 	1300 6150 1400 6150
@@
 	1800 6750 1800 6150
 Text GLabel 3550 5250 2    59   Input ~ 12
-FilterOut
+FilterOut2
 Wire Wire Line
 	3550 5650 3550 5250
@@
 Connection ~ 1450 2900
 Text GLabel 1650 2800 2    59   Input ~ 12
-LP
+LP2
 Text GLabel 1650 1950 2    59   Input ~ 12
-HP
+HP2
 Text GLabel 1650 2350 2    59   Input ~ 12
-BP
+BP2
 Wire Wire Line
 	1300 1950 1650 1950
@@
 	1450 3350 1450 3550
 Text GLabel 1650 3650 2    59   Input ~ 12
-CV
+CV2
 Text GLabel 1650 3250 2    59   Input ~ 12
-Out
+Out2
 Wire Wire Line
 	1300 3250 1650 3250
@@
 $EndComp
 Text GLabel 2550 2500 0    59   Input ~ 12
-FilterOut
+FilterOut2
 Wire Wire Line
 	2950 2500 2850 2500
@@
 	3600 2300 3600 2200
 Text GLabel 4400 3450 3    59   Input ~ 12
-BP
+BP2
 $Comp
 L Device:R R?
@@
 	4400 2600 4400 2400
 Text GLabel 5000 2600 2    59   Input ~ 12
-Out
+Out2
 Wire Wire Line
 	4800 2600 5000 2600
@@
 AR Path="/5C4E0953/5C59B140" Ref="C205"  Part="1"
 F 0 "C205" V 1355 1400 50  0000 C CNN
-F 1 "CP" V 1264 1400 50  0000 C CNN
+F 1 "100uF" V 1264 1400 50  0000 C CNN
 F 2 "Capacitor_Tantalum_SMD:CP_EIA-7343-15_Kemet-W_Pad2.25x2.55mm_HandSolder" H 1138 1250 50  0001 C CNN
 F 3 "~" H 1100 1400 50  0001 C CNN
@@
 $EndComp
 Wire Wire Line
-	3550 900  3900 900
+	3550 900  3700 900
+$Comp
+L power:PWR_FLAG #FLG0105
+U 1 1 5C60E2C0
+P 3700 750
+F 0 "#FLG0105" H 3700 825 50  0001 C CNN
+F 1 "PWR_FLAG" H 3700 924 50  0000 C CNN
+F 2 "" H 3700 750 50  0001 C CNN
+F 3 "~" H 3700 750 50  0001 C CNN
+	1    3700 750
+	1    0    0    -1
+$EndComp
+Wire Wire Line
+	3700 750  3700 900
+Connection ~ 3700 900
+Wire Wire Line
+	3700 900  3900 900
 $EndSCHEMATC
