File: Kicad_JE_SteinerVCF/JE-VCO1.sch (KiCad schematic (older format))
At the start: 56 parts, among them J301 Sine, J302 Tri, J303 Sq, J304 CV, J305 CV, P301 Doepfer_Power_10pin, U301 TL074, U302 ICL8038

Commit message: VCO inspiration
Parts:
- RV301: value 10k -> 10k Sin
- RV302: value 10k -> 10k Tri
- RV303: value 100k -> 100k Duty
- RV305: value 10k -> 10k SQ
- RV309: value 100k -> 100k CV
- RV310: value 100k -> 100k Coarse
- RV311: value 100k -> 100k fine
Changed lines of the file:
@@
 P 7875 2150
 F 0 "RV301" H 7805 2196 50  0000 R CNN
-F 1 "10k" H 7805 2105 50  0000 R CNN
+F 1 "10k Sin" H 7805 2105 50  0000 R CNN
 F 2 "Potentiometer_THT:Potentiometer_Alps_RK09K_Single_Vertical" H 7875 2150 50  0001 C CNN
 F 3 "~" H 7875 2150 50  0001 C CNN
@@
 P 5700 2250
 F 0 "RV302" H 5630 2296 50  0000 R CNN
-F 1 "10k" H 5630 2205 50  0000 R CNN
+F 1 "10k Tri" H 5630 2205 50  0000 R CNN
 F 2 "Potentiometer_THT:Potentiometer_Alps_RK09K_Single_Vertical" H 5700 2250 50  0001 C CNN
 F 3 "~" H 5700 2250 50  0001 C CNN
@@
 P 10425 3700
 F 0 "RV305" H 10355 3746 50  0000 R CNN
-F 1 "10k" H 10355 3655 50  0000 R CNN
+F 1 "10k SQ" H 10355 3655 50  0000 R CNN
 F 2 "Potentiometer_THT:Potentiometer_Alps_RK09K_Single_Vertical" H 10425 3700 50  0001 C CNN
 F 3 "~" H 10425 3700 50  0001 C CNN
@@
 P 5900 5575
 F 0 "RV311" V 5786 5575 50  0000 C CNN
-F 1 "100k" V 5695 5575 50  0000 C CNN
+F 1 "100k fine" V 5695 5575 50  0000 C CNN
 F 2 "Potentiometer_THT:Potentiometer_Alps_RK09K_Single_Vertical" H 5900 5575 50  0001 C CNN
 F 3 "~" H 5900 5575 50  0001 C CNN
@@
 P 4950 5575
 F 0 "RV310" V 4836 5575 50  0000 C CNN
-F 1 "100k" V 4745 5575 50  0000 C CNN
+F 1 "100k Coarse" V 4745 5575 50  0000 C CNN
 F 2 "Potentiometer_THT:Potentiometer_Alps_RK09K_Single_Vertical" H 4950 5575 50  0001 C CNN
 F 3 "~" H 4950 5575 50  0001 C CNN
@@
 P 4050 4850
 F 0 "RV309" H 3980 4896 50  0000 R CNN
-F 1 "100k" H 3980 4805 50  0000 R CNN
+F 1 "100k CV" H 3980 4805 50  0000 R CNN
 F 2 "Potentiometer_THT:Potentiometer_Alps_RK09K_Single_Vertical" H 4050 4850 50  0001 C CNN
 F 3 "~" H 4050 4850 50  0001 C CNN
@@
 P 8375 3000
 F 0 "RV303" H 8305 2954 50  0000 R CNN
-F 1 "100k" H 8305 3045 50  0000 R CNN
+F 1 "100k Duty" H 8305 3045 50  0000 R CNN
 F 2 "Potentiometer_THT:Potentiometer_Alps_RK09K_Single_Vertical" H 8375 3000 50  0001 C CNN
 F 3 "~" H 8375 3000 50  0001 C CNN
