File: Kicad_JE_SteinerVCF - RevB/JE-VCO1.sch (KiCad schematic (older format))
At the start: 50 parts, among them J301 Sine, J302 Tri, J303 Sq, J305 CV, P301 Doepfer_Power_10pin, U301 TL074, U302 ICL8038

Commit message: VCF SMD routed
Parts:
- C302, C304: footprint Capacitor_THT:CP_Radial_D10.0mm_P5.00mm -> Capacitor_SMD:C_1206_3216Metric
- D302: footprint Diode_SMD:D_SOD-123 -> Diode_SMD:D_MiniMELF
- RV301, RV302, RV303, RV305, RV307, RV309, RV310, RV311: footprint Potentiometer_THT:Potentiometer_Alps_RK09K_Single_Vertical -> AJ:Potentiometer_China_RK09_Single_Vertical_AJ
Changed lines of the file:
@@
 F 0 "C302" H 3093 896 50  0000 L CNN
 F 1 "100u" H 3093 805 50  0000 L CNN
-F 2 "Capacitor_THT:CP_Radial_D10.0mm_P5.00mm" H 3013 700 50  0001 C CNN
+F 2 "Capacitor_SMD:C_1206_3216Metric" H 3013 700 50  0001 C CNN
 F 3 "~" H 2975 850 50  0001 C CNN
 	1    2975 850
@@
 F 0 "C304" H 3093 1196 50  0000 L CNN
 F 1 "100u" H 3093 1105 50  0000 L CNN
-F 2 "Capacitor_THT:CP_Radial_D10.0mm_P5.00mm" H 3013 1000 50  0001 C CNN
+F 2 "Capacitor_SMD:C_1206_3216Metric" H 3013 1000 50  0001 C CNN
 F 3 "~" H 2975 1150 50  0001 C CNN
 	1    2975 1150
@@
 F 0 "RV301" H 7805 2196 50  0000 R CNN
 F 1 "50k Sin" H 7805 2105 50  0000 R CNN
-F 2 "Potentiometer_THT:Potentiometer_Alps_RK09K_Single_Vertical" H 7875 2150 50  0001 C CNN
+F 2 "AJ:Potentiometer_China_RK09_Single_Vertical_AJ" H 7875 2150 50  0001 C CNN
 F 3 "~" H 7875 2150 50  0001 C CNN
 	1    7875 2150
@@
 F 0 "RV302" H 5630 2296 50  0000 R CNN
 F 1 "50k Tri" H 5630 2205 50  0000 R CNN
-F 2 "Potentiometer_THT:Potentiometer_Alps_RK09K_Single_Vertical" H 5700 2250 50  0001 C CNN
+F 2 "AJ:Potentiometer_China_RK09_Single_Vertical_AJ" H 5700 2250 50  0001 C CNN
 F 3 "~" H 5700 2250 50  0001 C CNN
 	1    5700 2250
@@
 F 0 "RV305" H 10900 3450 50  0000 R CNN
 F 1 "50k SQ" H 10950 3525 50  0000 R CNN
-F 2 "Potentiometer_THT:Potentiometer_Alps_RK09K_Single_Vertical" H 10575 3700 50  0001 C CNN
+F 2 "AJ:Potentiometer_China_RK09_Single_Vertical_AJ" H 10575 3700 50  0001 C CNN
 F 3 "~" H 10575 3700 50  0001 C CNN
 	1    10575 3700
@@
 F 0 "RV311" V 5786 5575 50  0000 C CNN
 F 1 "100k fine" V 5695 5575 50  0000 C CNN
-F 2 "Potentiometer_THT:Potentiometer_Alps_RK09K_Single_Vertical" H 5900 5575 50  0001 C CNN
+F 2 "AJ:Potentiometer_China_RK09_Single_Vertical_AJ" H 5900 5575 50  0001 C CNN
 F 3 "~" H 5900 5575 50  0001 C CNN
 	1    5900 5575
@@
 F 0 "RV310" V 4836 5575 50  0000 C CNN
 F 1 "100k Coarse" V 4745 5575 50  0000 C CNN
-F 2 "Potentiometer_THT:Potentiometer_Alps_RK09K_Single_Vertical" H 4950 5575 50  0001 C CNN
+F 2 "AJ:Potentiometer_China_RK09_Single_Vertical_AJ" H 4950 5575 50  0001 C CNN
 F 3 "~" H 4950 5575 50  0001 C CNN
 	1    4950 5575
@@
 F 0 "RV309" H 3005 4896 50  0000 R CNN
 F 1 "100k CV" H 3005 4805 50  0000 R CNN
-F 2 "Potentiometer_THT:Potentiometer_Alps_RK09K_Single_Vertical" H 3075 4850 50  0001 C CNN
+F 2 "AJ:Potentiometer_China_RK09_Single_Vertical_AJ" H 3075 4850 50  0001 C CNN
 F 3 "~" H 3075 4850 50  0001 C CNN
 	1    3075 4850
@@
 F 0 "D302" H 7450 5067 50  0000 C CNN
 F 1 "MMSD4148" H 7450 4976 50  0000 C CNN
-F 2 "Diode_SMD:D_SOD-123" H 7450 4675 50  0001 C CNN
+F 2 "Diode_SMD:D_MiniMELF" H 7450 4675 50  0001 C CNN
 F 3 "https://www.onsemi.com/pub/Collateral/MMSD4148T1-D.PDF" H 7450 4850 50  0001 C CNN
 	1    7450 4850
@@
 F 0 "RV303" H 8380 2779 50  0000 R CNN
 F 1 "100k Duty" H 8380 2870 50  0000 R CNN
-F 2 "Potentiometer_THT:Potentiometer_Alps_RK09K_Single_Vertical" H 8450 2825 50  0001 C CNN
+F 2 "AJ:Potentiometer_China_RK09_Single_Vertical_AJ" H 8450 2825 50  0001 C CNN
 F 3 "~" H 8450 2825 50  0001 C CNN
 	1    8450 2825
@@
 F 0 "RV307" H 3705 5146 50  0000 R CNN
 F 1 "100k Glide" H 3705 5055 50  0000 R CNN
-F 2 "Potentiometer_THT:Potentiometer_Alps_RK09K_Single_Vertical" H 3775 5100 50  0001 C CNN
+F 2 "AJ:Potentiometer_China_RK09_Single_Vertical_AJ" H 3775 5100 50  0001 C CNN
 F 3 "~" H 3775 5100 50  0001 C CNN
 	1    3775 5100
