File: Kicad_JE_SteinerVCF - RevB/JE-SMD-SteinerVCF.sch (KiCad schematic (older format))
At the start: 58 parts, among them J201 HP, J202 BP, J203 LP, J204 Out, J205 CV, P201 Doepfer_Power_10pin, Q201 MMBT2907A, Q202 MMBT2222A, Q203 MMBT2222A, Q204 MMBT2222A

Commit message: Gerber
Parts:
- RV202, RV203: footprint AJ-Dropbox-Kicad:AlpsRK09K -> AJ-Dropbox-Kicad:Potentiometer_China_RK09_Single_Vertical_AJ
- gave numbers to parts that had none: 1
Changed lines of the file:
@@
 F 0 "RV203" H 1205 6796 50  0000 R CNN
 F 1 "100k" H 1205 6705 50  0000 R CNN
-F 2 "AJ-Dropbox-Kicad:AlpsRK09K" H 1275 6750 50  0001 C CNN
+F 2 "AJ-Dropbox-Kicad:Potentiometer_China_RK09_Single_Vertical_AJ" H 1275 6750 50  0001 C CNN
 F 3 "~" H 1275 6750 50  0001 C CNN
 	1    1275 6750
@@
 F 0 "RV202" H 1105 5846 50  0000 R CNN
 F 1 "100k" H 1105 5755 50  0000 R CNN
-F 2 "AJ-Dropbox-Kicad:AlpsRK09K" H 1175 5800 50  0001 C CNN
+F 2 "AJ-Dropbox-Kicad:Potentiometer_China_RK09_Single_Vertical_AJ" H 1175 5800 50  0001 C CNN
 F 3 "~" H 1175 5800 50  0001 C CNN
 	1    1175 5800
@@
 P 3700 7150
 AR Path="/5DF41AC2" Ref="C?"  Part="1"
-AR Path="/5C4E0953/5DF41AC2" Ref="C?"  Part="1"
-F 0 "C?" V 3448 7150 50  0000 C CNN
+AR Path="/5C4E0953/5DF41AC2" Ref="C216"  Part="1"
+F 0 "C216" V 3448 7150 50  0000 C CNN
 F 1 "22u" V 3539 7150 50  0000 C CNN
 F 2 "Capacitor_SMD:C_0805_2012Metric_Pad1.15x1.40mm_HandSolder" H 3738 7000 50  0001 C CNN
