File: Kicad_JE_SteinerVCF - RevB/Kicad_JE_SteinerVCF.sch (KiCad schematic (older format))
At the start: 74 parts, among them J101 HP, J102 BP, J103 LP, J104 Out, J105 CV, J106 CV, P101 Doepfer_Power_10pin, Q101 BC559, Q102 BC549, Q103 BC549, Q104 BC549, Q105 BC549, Q106 BC549

Commit message: VCF SMD routed
Parts:
- RV101, RV102, RV103, RV104: footprint Potentiometer_THT:Potentiometer_Alps_RK09K_Single_Vertical -> AJ:Potentiometer_China_RK09_Single_Vertical_AJ
Changed lines of the file:
@@
 F 0 "RV101" V 5393 3000 50  0000 C CNN
 F 1 "5k" V 5484 3000 50  0000 C CNN
-F 2 "Potentiometer_THT:Potentiometer_Alps_RK09K_Single_Vertical" H 5600 3000 50  0001 C CNN
+F 2 "AJ:Potentiometer_China_RK09_Single_Vertical_AJ" H 5600 3000 50  0001 C CNN
 F 3 "~" H 5600 3000 50  0001 C CNN
 	1    5600 3000
@@
 F 0 "RV103" H 2230 7121 50  0000 R CNN
 F 1 "100k" H 2230 7030 50  0000 R CNN
-F 2 "Potentiometer_THT:Potentiometer_Alps_RK09K_Single_Vertical" H 2300 7075 50  0001 C CNN
+F 2 "AJ:Potentiometer_China_RK09_Single_Vertical_AJ" H 2300 7075 50  0001 C CNN
 F 3 "~" H 2300 7075 50  0001 C CNN
 	1    2300 7075
@@
 F 0 "RV104" V 1943 6150 50  0000 C CNN
 F 1 "100k" V 2034 6150 50  0000 C CNN
-F 2 "Potentiometer_THT:Potentiometer_Alps_RK09K_Single_Vertical" H 2150 6150 50  0001 C CNN
+F 2 "AJ:Potentiometer_China_RK09_Single_Vertical_AJ" H 2150 6150 50  0001 C CNN
 F 3 "~" H 2150 6150 50  0001 C CNN
 	1    2150 6150
@@
 F 0 "RV102" V 1943 5525 50  0000 C CNN
 F 1 "100k" V 2034 5525 50  0000 C CNN
-F 2 "Potentiometer_THT:Potentiometer_Alps_RK09K_Single_Vertical" H 2150 5525 50  0001 C CNN
+F 2 "AJ:Potentiometer_China_RK09_Single_Vertical_AJ" H 2150 5525 50  0001 C CNN
 F 3 "~" H 2150 5525 50  0001 C CNN
 	1    2150 5525

Commit message: Gerber
Parts:
- C102, C103, C105, C111: footprint Capacitor_THT:CP_Radial_D10.0mm_P5.00mm -> Capacitor_THT:C_Radial_D8.0mm_H7.0mm_P3.50mm
- C107: footprint Capacitor_THT:CP_Radial_D10.0mm_P3.80mm -> Capacitor_THT:C_Radial_D8.0mm_H7.0mm_P3.50mm
- C113, C116: footprint Capacitor_THT:C_Rect_L7.0mm_W2.0mm_P5.00mm -> Capacitor_THT:C_Radial_D8.0mm_H7.0mm_P3.50mm
Changed lines of the file:
@@
 F 0 "C102" H 5818 1146 50  0000 L CNN
 F 1 "CP" H 5818 1055 50  0000 L CNN
-F 2 "Capacitor_THT:CP_Radial_D10.0mm_P5.00mm" H 5738 950 50  0001 C CNN
+F 2 "Capacitor_THT:C_Radial_D8.0mm_H7.0mm_P3.50mm" H 5738 950 50  0001 C CNN
 F 3 "~" H 5700 1100 50  0001 C CNN
 	1    5700 1100
@@
 F 0 "C103" H 6368 1146 50  0000 L CNN
 F 1 "100u" H 6368 1055 50  0000 L CNN
-F 2 "Capacitor_THT:CP_Radial_D10.0mm_P5.00mm" H 6288 950 50  0001 C CNN
+F 2 "Capacitor_THT:C_Radial_D8.0mm_H7.0mm_P3.50mm" H 6288 950 50  0001 C CNN
 F 3 "~" H 6250 1100 50  0001 C CNN
 	1    6250 1100
@@
 F 0 "C111" H 4768 7196 50  0000 L CNN
 F 1 "100u" H 4768 7105 50  0000 L CNN
-F 2 "Capacitor_THT:CP_Radial_D10.0mm_P5.00mm" H 4688 7000 50  0001 C CNN
+F 2 "Capacitor_THT:C_Radial_D8.0mm_H7.0mm_P3.50mm" H 4688 7000 50  0001 C CNN
 F 3 "~" H 4650 7150 50  0001 C CNN
 	1    4650 7150
@@
 F 0 "C107" V 6305 2650 50  0000 C CNN
 F 1 "10u" V 6214 2650 50  0000 C CNN
-F 2 "Capacitor_THT:CP_Radial_D10.0mm_P3.80mm" H 6088 2500 50  0001 C CNN
+F 2 "Capacitor_THT:C_Radial_D8.0mm_H7.0mm_P3.50mm" H 6088 2500 50  0001 C CNN
 F 3 "~" H 6050 2650 50  0001 C CNN
 	1    6050 2650
@@
 F 0 "C105" V 4105 1350 50  0000 C CNN
 F 1 "CP" V 4014 1350 50  0000 C CNN
-F 2 "Capacitor_THT:CP_Radial_D10.0mm_P5.00mm" H 3888 1200 50  0001 C CNN
+F 2 "Capacitor_THT:C_Radial_D8.0mm_H7.0mm_P3.50mm" H 3888 1200 50  0001 C CNN
 F 3 "~" H 3850 1350 50  0001 C CNN
 	1    3850 1350
@@
 F 0 "C116" V 2648 3325 50  0000 C CNN
 F 1 "10u" V 2739 3325 50  0000 C CNN
-F 2 "Capacitor_THT:C_Rect_L7.0mm_W2.0mm_P5.00mm" H 2938 3175 50  0001 C CNN
+F 2 "Capacitor_THT:C_Radial_D8.0mm_H7.0mm_P3.50mm" H 2938 3175 50  0001 C CNN
 F 3 "~" H 2900 3325 50  0001 C CNN
 	1    2900 3325
@@
 F 0 "C113" V 2523 1650 50  0000 C CNN
 F 1 "10u" V 2614 1650 50  0000 C CNN
-F 2 "Capacitor_THT:C_Rect_L7.0mm_W2.0mm_P5.00mm" H 2813 1500 50  0001 C CNN
+F 2 "Capacitor_THT:C_Radial_D8.0mm_H7.0mm_P3.50mm" H 2813 1500 50  0001 C CNN
 F 3 "~" H 2775 1650 50  0001 C CNN
 	1    2775 1650
